File: STLINKV2-1/STLINKV2-1.sch (KiCad schematic (older format))
At the start: 47 parts, among them J1 USB_A, J2 Conn_01x04, J3 Top, J4 Buttom, J5 Conn_01x02, Q1 MMBT5551L, U1 TLV73333PDBV, U2 STM32F103C8Tx, Y1 8M

Commit message: layout 基本完成
Parts:
- J2: footprint (none) -> Connector_PinSocket_2.54mm:PinSocket_1x04_P2.54mm_Vertical
- J5: footprint (none) -> Connector_PinSocket_2.54mm:PinSocket_1x02_P2.54mm_Vertical
Connections:
- net +3V3: now also J4.2 (Pin_2); no longer J4.4 (Pin_4)
- net +5V: now also J4.1 (Pin_1); no longer J4.5 (Pin_5)
- net P_SWCLK: now also J4.5 (Pin_5); no longer J4.1 (Pin_1)
- net P_SWDIO: now also J4.4 (Pin_4); no longer J4.2 (Pin_2)
Changed lines of the file:
@@
 F 3 "~" H 10300 6000 50  0001 C CNN
 	1    10300 6000
-	1    0    0    1
+	1    0    0    -1
 $EndComp
 $Comp
@@
 F 0 "J2" H 9055 5642 50  0000 L CNN
 F 1 "Conn_01x04" H 9055 5551 50  0000 L CNN
-F 2 "" H 8975 5650 50  0001 C CNN
+F 2 "Connector_PinSocket_2.54mm:PinSocket_1x04_P2.54mm_Vertical" H 8975 5650 50  0001 C CNN
 F 3 "~" H 8975 5650 50  0001 C CNN
 	1    8975 5650
@@
 F 0 "J5" H 9055 6042 50  0000 L CNN
 F 1 "Conn_01x02" H 9055 5951 50  0000 L CNN
-F 2 "" H 8975 6050 50  0001 C CNN
+F 2 "Connector_PinSocket_2.54mm:PinSocket_1x02_P2.54mm_Vertical" H 8975 6050 50  0001 C CNN
 F 3 "~" H 8975 6050 50  0001 C CNN
 	1    8975 6050
